File: Guide68/Top_L/Guide68_Top_L.kicad_pcb (KiCad board)
At the start: 2 copper layers, 133.3 x 95.2 mm, 33 parts, among them SW1 SW_PUSH, SW10 SW_PUSH, SW11 SW_PUSH, SW12 SW_PUSH, SW13 SW_PUSH, SW14 SW_PUSH, SW15 SW_PUSH, SW16 SW_PUSH, SW17 SW_PUSH, SW18 SW_PUSH, SW19 SW_PUSH, SW2 SW_PUSH, SW20 SW_PUSH, SW21 SW_PUSH, SW22 SW_PUSH, SW23 SW_PUSH, SW24 SW_PUSH, SW25 SW_PUSH, SW26 SW_PUSH, SW27 SW_PUSH, SW28 SW_PUSH, SW29 SW_PUSH, SW3 SW_PUSH, SW4 SW_PUSH, SW5 SW_PUSH, SW6 SW_PUSH, SW7 SW_PUSH, SW8 SW_PUSH, SW9 SW_PUSH

Commit message: スイッチ穴を更新
Parts:
- Ref** (x4): footprint kbd_Hole:m2_Screw_Hole -> kbd_Hole_Public:m2_Screw_Hole
- SW1, SW10, SW11, SW12, SW13, SW14, SW15, SW16, SW17, SW18, SW19, SW2, SW20, SW21, SW22, SW23, SW24, SW25, SW26, SW27, SW28, SW29, SW3, SW5, SW6, SW7, SW8, SW9: footprint kbd_SW_Hole:SW_Hole_TH_1u_fix -> kbd_SW_Hole_Public:SW_Hole_TH_1u
- SW4: footprint kbd_SW_Hole:SW_Hole_TH_2.25u_fix -> kbd_SW_Hole_Public:SW_Hole_TH_2u
