File: Guide68/Top_R/Guide68_Top_R.kicad_pcb (KiCad board)
At the start: 2 copper layers, 171.5 x 95.2 mm, 45 parts, among them J13 Conn_01x01, J14 Conn_01x01, J15 Conn_01x01, J16 Conn_01x01, J4 Conn_01x01, J5 Conn_01x01, SW30 SW_PUSH, SW31 SW_PUSH, SW32 SW_PUSH, SW33 SW_PUSH, SW34 SW_PUSH, SW35 SW_PUSH, SW36 SW_PUSH, SW37 SW_PUSH, SW38 SW_PUSH, SW39 SW_PUSH, SW40 SW_PUSH, SW41 SW_PUSH, SW42 SW_PUSH, SW43 SW_PUSH, SW44 SW_PUSH, SW45 SW_PUSH, SW46 SW_PUSH, SW47 SW_PUSH, SW48 SW_PUSH, SW49 SW_PUSH, SW50 SW_PUSH, SW51 SW_PUSH, SW52 SW_PUSH, SW53 SW_PUSH, SW54 SW_PUSH, SW55 SW_PUSH, SW56 SW_PUSH, SW57 SW_PUSH, SW58 SW_PUSH, SW59 SW_PUSH, SW60 SW_PUSH, SW61 SW_PUSH, SW62 SW_PUSH, SW63 SW_PUSH, SW64 SW_PUSH, SW65 SW_PUSH, SW66 SW_PUSH, SW67 SW_PUSH, SW68 SW_PUSH

Commit message: スイッチ穴を更新
Parts:
- J13, J14, J15, J16, J4, J5: footprint kbd_Hole:m2_Screw_Hole -> kbd_Hole_Public:m2_Screw_Hole
- SW30, SW31, SW32, SW33, SW34, SW35, SW36, SW37, SW38, SW39, SW40, SW41, SW42, SW43, SW44, SW45, SW46, SW47, SW48, SW49, SW50, SW51, SW52, SW53, SW54, SW55, SW56, SW57, SW58, SW59, SW60, SW62, SW63, SW64, SW65, SW66, SW67, SW68: footprint kbd_SW_Hole:SW_Hole_TH_1u_fix -> kbd_SW_Hole_Public:SW_Hole_TH_1u
- SW61: footprint kbd_SW_Hole:SW_Hole_TH_2.25u_fix -> kbd_SW_Hole_Public:SW_Hole_TH_2.25u
